Commit message: update wsg xacro

File: wsg_32_description/robots/wsg_32_description.urdf.xacro (robot description, xacro)
@@ -260,4 +260,37 @@
     <child link="${name}_left_gelsight_finger_link" />
   </joint>
+  <link
+    name="${name}_left_gelsight_finger_pad">
+  </link>
+  <joint
+    name="${name}_left_gelsight_finger_pad_joint"
+    type="fixed">
+    <origin
+      xyz="0 0.0742 0"/>
+    <parent link="${name}_left_gelsight_finger_link" />
+    <child link="${name}_left_gelsight_finger_pad" />
+  </joint>
+  <link
+    name="${name}_right_gelsight_finger_pad">
+  </link>
+  <joint
+    name="${name}_right_gelsight_finger_pad_joint"
+    type="fixed">
+    <origin
+      xyz="0 0.0742 0"/>
+    <parent link="${name}_right_gelsight_finger_link" />
+    <child link="${name}_right_gelsight_finger_pad" />
+  </joint>
+  <link
+    name="${name}_grasp_link">
+  </link>
+  <joint
+    name="${name}_grasp_link_jnt"
+    type="fixed">
+    <origin
+      xyz="0 0 0.1512"/>
+    <parent link="${name}_base_link" />
+    <child link="{name}_grasp_link" />
+  </joint>
 </xacro:macro>
 </robot>
