Commit message: new dual arm moveit config and working dual arm controller

File: dual_mars_arm_moveit_config/config/dual_mars_arm.srdf.xacro (robot description, xacro)
@@ -7,7 +7,7 @@
   <xacro:arg name="arm_1_id" default="pan_pan"/>
   <xacro:arg name="arm_2_id" default="an_an"/>
-  <xacro:include filename="$(find dual_mars_arm_moveit_config)/config/panda_arm_hand.xacro" />
-  <xacro:panda_arm_hand prefix="$(arg arm_1_id)"/>
-  <xacro:panda_arm_hand prefix="$(arg arm_2_id)"/>
+  <xacro:include filename="$(find dual_mars_arm_moveit_config)/config/panda_arm.xacro" />
+  <xacro:panda_arm prefix="$(arg arm_1_id)"/>
+  <xacro:panda_arm prefix="$(arg arm_2_id)"/>
   <!--GROUPS: Representation of a set of joints and links. This can be useful for specifying DOF to plan for, defining arms, end effectors, etc-->
   <!--LINKS: When a link is specified, the parent joint of that link (if it exists) is automatically included-->
@@ -15,8 +15,25 @@
   <!--CHAINS: When a chain is specified, all the links along the chain (including endpoints) are included in the group. Additionally, all the joints that are parents to included links are also included. This means that joints along the chain and the parent joint of the base link are included in the group-->
   <!--SUBGROUPS: Groups can also be formed by referencing to already defined group names-->
-  <group name="$(arg arm_1_id)_and_$(arg arm_2_id)">
-      <group name="$(arg arm_1_id)_arm_hand"/>
-      <group name="$(arg arm_2_id)_arm_hand"/>
+  <group name="combined_arms">
+      <group name="$(arg arm_1_id)_arm"/>
+      <group name="$(arg arm_2_id)_arm"/>
   </group>
+  <group_state name="ready" group="combined_arms">
+    <joint name="$(arg arm_1_id)_joint1" value="0" />
+    <joint name="$(arg arm_1_id)_joint2" value="-0.785" />
+    <joint name="$(arg arm_1_id)_joint3" value="0" />
+    <joint name="$(arg arm_1_id)_joint4" value="-2.356" />
+    <joint name="$(arg arm_1_id)_joint5" value="0" />
+    <joint name="$(arg arm_1_id)_joint6" value="1.571" />
+    <joint name="$(arg arm_1_id)_joint7" value="0.785" />
+    <joint name="$(arg arm_2_id)_joint1" value="0" />
+    <joint name="$(arg arm_2_id)_joint2" value="-0.785" />
+    <joint name="$(arg arm_2_id)_joint3" value="0" />
+    <joint name="$(arg arm_2_id)_joint4" value="-2.356" />
+    <joint name="$(arg arm_2_id)_joint5" value="0" />
+    <joint name="$(arg arm_2_id)_joint6" value="1.571" />
+    <joint name="$(arg arm_2_id)_joint7" value="0.785" />
+  </group_state>
+  <virtual_joint name="world_to_arm" type="fixed" parent_frame="world" child_link="base" />
   <!--DISABLE COLLISIONS: By default it is assumed that any link of the robot could potentially come into collision with any other link in the robot. This tag disables collision checking between a specified pair of links. -->
   <disable_collisions link1="base" link2="$(arg arm_1_id)_link0" reason="Adjacent"/>

File: franka_description/robots/dual_mars_arm.urdf.xacro (robot description, xacro)
@@ -10,5 +10,5 @@
       <origin xyz="0 0 0.5" rpy="0 0 0"/>
       <geometry>
-        <box size="1 2 1" />
+        <box size="1.5 2 1" />
       </geometry>
       <material name="White">
@@ -19,13 +19,11 @@
       <origin xyz="0 0 0.5" rpy="0 0 0"/>
       <geometry>
-        <box size="1 2 1" />
+        <box size="1.5 2 1" />
       </geometry>
     </collision>
   </link>
-  <!-- right arm with gripper -->
-  <xacro:panda_arm arm_id="$(arg an_an_id)" connected_to="base"  xyz="0 -0.5 1" safety_distance="0.03"/>
-  <xacro:hand arm_id="$(arg an_an_id)" rpy="0 0 ${-pi/4}" connected_to="$(arg an_an_id)_link8" safety_distance="0.03"/>
-  <!-- left arm with gripper -->
-  <xacro:panda_arm arm_id="$(arg pan_pan_id)" connected_to="base"  xyz="0 0.5 1" safety_distance="0.03"/>
-  <xacro:hand arm_id="$(arg pan_pan_id)" rpy="0 0 ${-pi/4}" connected_to="$(arg pan_pan_id)_link8" safety_distance="0.03"/>
+  <xacro:panda_arm arm_id="$(arg pan_pan_id)" connected_to="base"  xyz="-0.2336 -0.515 1"  safety_distance="0.005"/>
+  <!-- <xacro:hand arm_id="$(arg pan_pan_id)" rpy="0 0 ${-pi/4}" connected_to="$(arg pan_pan_id)_link8" safety_distance="0.005"/> -->
+  <xacro:panda_arm arm_id="$(arg an_an_id)" connected_to="base"  xyz="0.2336 0.515 1" rpy="0 0 ${-pi}" safety_distance="0.005"/>
+  <!-- <xacro:hand arm_id="$(arg an_an_id)" rpy="0 0 ${-pi/4}" connected_to="$(arg an_an_id)_link8" safety_distance="0.005"/> -->
 </robot>

Commit message: updated dual arm,  wsg urdf/srdf

File: dual_mars_arm_moveit_config/config/dual_mars_arm.srdf.xacro (robot description, xacro)
@@ -47,16 +47,4 @@
   <disable_collisions link1="base" link2="$(arg arm_2_id)_link3" reason="Never"/>
   <disable_collisions link1="base" link2="$(arg arm_2_id)_link4" reason="Never"/>
-  <disable_collisions link1="an_an_link7" link2=" wsg_an_an_base_link" reason="Adjacent"/>
-<disable_collisions link1="base" link2="camera_mount" reason="Adjacent"/>
-<disable_collisions link1="pan_pan_link7" link2="wsg_pan_pan_base_link"/>
-<disable_collisions link1="wsg_an_an_base_link" link2="wsg_an_an_base_link_gripper_left"/>
-<disable_collisions link1="wsg_an_an_base_link" link2="wsg_an_an_base_link_gripper_right"/>
-<disable_collisions link1="wsg_an_an_base_link_gripper_left" link2="wsg_an_an_base_link_gripper_right"/>
-<disable_collisions link1="wsg_an_an_base_link_gripper_left" link2="wsg_an_an_left_gelsight_finger_link"/>
-<disable_collisions link1="wsg_an_an_base_link_gripper_right" link2="wsg_an_an_right_gelsight_finger_link"/>
-<disable_collisions link1="wsg_pan_pan_base_link" link2="wsg_pan_pan_base_link_gripper_left"/>
-<disable_collisions link1="wsg_pan_pan_base_link" link2="wsg_pan_pan_base_link_gripper_right"/>
-<disable_collisions link1="wsg_pan_pan_base_link_gripper_left" link2="wsg_pan_pan_base_link_gripper_right"/>
-<disable_collisions link1="wsg_pan_pan_base_link_gripper_left" link2="wsg_pan_pan_left_gelsight_finger_link"/>
-<disable_collisions link1="wsg_pan_pan_base_link_gripper_right" link2="wsg_pan_pan_right_gelsight_finger_link"/>
+  <disable_collisions link1="base" link2="camera_mount" reason="Adjacent"/>
 </robot>

File: dual_mars_arm_moveit_config/config/panda_arm.xacro (robot description, xacro)
@@ -60,4 +60,11 @@
     <disable_collisions link1="${prefix}_link6" link2="${prefix}_link8" reason="Default" />
     <disable_collisions link1="${prefix}_link7" link2="${prefix}_link8" reason="Adjacent" />
+    <disable_collisions link1="${prefix}_wsg_base_link" link2="${prefix}_wsg_base_link_gripper_left"/>
+    <disable_collisions link1="${prefix}_wsg_base_link" link2="${prefix}_wsg_base_link_gripper_right"/>
+    <disable_collisions link1="${prefix}_wsg_base_link_gripper_left" link2="${prefix}_wsg_base_link_gripper_right"/>
+    <disable_collisions link1="${prefix}_wsg_base_link_gripper_left" link2="${prefix}_wsg_left_gelsight_finger_link"/>
+    <disable_collisions link1="${prefix}_wsg_base_link_gripper_right" link2="${prefix}_wsg_right_gelsight_finger_link"/>
+    <disable_collisions link1="${prefix}_link7" link2="${prefix}_wsg_base_link"/>
+    <disable_collisions link1="${prefix}_link8" link2="${prefix}_wsg_base_link"/>
   </xacro:macro>
 </robot>

File: franka_description/robots/dual_mars_arm.urdf.xacro (robot description, xacro)
@@ -24,9 +24,9 @@
     </collision>
   </link>
-  <xacro:panda_arm arm_id="$(arg pan_pan_id)" connected_to="base"  xyz="-0.2336 -0.515 1"  safety_distance="0.005"/>
+  <xacro:panda_arm arm_id="$(arg pan_pan_id)" connected_to="base"  xyz="-0.2301 -0.5065 0.995"  safety_distance="0.005"/>
   <!-- <xacro:hand arm_id="$(arg pan_pan_id)" rpy="0 0 ${-pi/4}" connected_to="$(arg pan_pan_id)_link8" safety_distance="0.005"/> -->
-  <xacro:wsg_32_xacro name="wsg_pan_pan" parent="$(arg pan_pan_id)_link8"  xyz="0 0 0.01" />
-  <xacro:panda_arm arm_id="$(arg an_an_id)" connected_to="base"  xyz="0.2336 0.515 1" rpy="0 0 ${-pi}" safety_distance="0.005"/>
-  <xacro:wsg_32_xacro name="wsg_an_an" parent="$(arg an_an_id)_link8"  xyz="0 0 0.01" />
+  <xacro:wsg_32_xacro name="$(arg pan_pan_id)_wsg" parent="$(arg pan_pan_id)_link8"  xyz="0 0 0.01" rpy="0 0 ${-pi/2}" />
+  <xacro:panda_arm arm_id="$(arg an_an_id)" connected_to="base"  xyz="0.2301 0.5065 1.005" rpy="0 0 ${-pi}" safety_distance="0.005"/>
+  <xacro:wsg_32_xacro name="$(arg an_an_id)_wsg" parent="$(arg an_an_id)_link8"  xyz="0 0 0.01" rpy="0 0 ${-pi/2}"/>
   <!-- <xacro:hand arm_id="$(arg an_an_id)" rpy="0 0 ${-pi/4}" connected_to="$(arg an_an_id)_link8" safety_distance="0.005"/> -->
   <link name="camera_mount">

File: franka_description/robots/panda_arm.urdf.xacro (robot description, xacro)
@@ -11,8 +11,15 @@
     <xacro:include filename="$(find franka_description)/robots/panda_arm.xacro" />
     <xacro:panda_arm arm_id="$(arg arm_id)" safety_distance="0.03"/>
+    <xacro:include filename="$(find wsg_32_description)/robots/wsg_32_description.urdf.xacro"/>
+    <xacro:wsg_32_xacro name="$(arg arm_id)_wsg" parent="$(arg arm_id)_link8"  xyz="0 0 0.01" rpy="0 0 -${pi/2}"/>
     <xacro:if value="$(arg hand)">
       <xacro:include filename="$(find franka_description)/robots/hand.xacro"/>
       <xacro:hand arm_id="$(arg arm_id)" rpy="0 0 ${-pi/4}" connected_to="$(arg arm_id)_link8" safety_distance="0.03"/>
     </xacro:if>
+    <link name="world" />
+    <joint name="world_joint" type="fixed">
+      <parent link="world" />
+      <child  link="$(arg arm_id)_link0" />
+    </joint>
   </xacro:unless>
   <xacro:if value="$(arg gazebo)">

File: panda_moveit_config/config/panda_arm.xacro (robot description, xacro)
@@ -61,4 +61,11 @@
     <disable_collisions link1="${prefix}_link6" link2="${prefix}_link8" reason="Default" />
     <disable_collisions link1="${prefix}_link7" link2="${prefix}_link8" reason="Adjacent" />
+    <disable_collisions link1="${prefix}_wsg_base_link" link2="${prefix}_wsg_base_link_gripper_left"/>
+    <disable_collisions link1="${prefix}_wsg_base_link" link2="${prefix}_wsg_base_link_gripper_right"/>
+    <disable_collisions link1="${prefix}_wsg_base_link_gripper_left" link2="${prefix}_wsg_base_link_gripper_right"/>
+    <disable_collisions link1="${prefix}_wsg_base_link_gripper_left" link2="${prefix}_wsg_left_gelsight_finger_link"/>
+    <disable_collisions link1="${prefix}_wsg_base_link_gripper_right" link2="${prefix}_wsg_right_gelsight_finger_link"/>
+    <disable_collisions link1="${prefix}_link7" link2="${prefix}_wsg_base_link"/>
+    <disable_collisions link1="${prefix}_link8" link2="${prefix}_wsg_base_link"/>
   </xacro:macro>
 </robot>

File: panda_moveit_config/config/panda_arm_hand.srdf.xacro (robot description, xacro)
@@ -33,3 +33,8 @@
   <disable_collisions link1="panda_link7" link2="panda_rightfinger" reason="Never" />
   <disable_collisions link1="panda_link8" link2="panda_rightfinger" reason="Never" />
+  <disable_collisions link1="panda_wsg_base_link" link2="panda_wsg_base_link_gripper_left"/>
+  <disable_collisions link1="panda_wsg_base_link" link2="panda_wsg_base_link_gripper_right"/>
+  <disable_collisions link1="panda_wsg_base_link_gripper_left" link2="panda_wsg_base_link_gripper_right"/>
+  <disable_collisions link1="panda_wsg_base_link_gripper_left" link2="panda_wsg_left_gelsight_finger_link"/>
+  <disable_collisions link1="panda_wsg_base_link_gripper_right" link2="panda_wsg_right_gelsight_finger_link"/>
 </robot>

File: wsg_32_description/robots/wsg_32_description.urdf.xacro (robot description, xacro)
@@ -291,5 +291,5 @@
       xyz="0 0 0.1512"/>
     <parent link="${name}_base_link" />
-    <child link="{name}_grasp_link" />
+    <child link="${name}_grasp_link" />
   </joint>
 </xacro:macro>
