Commit message: added camera mount

File: franka_description/robots/dual_mars_arm.urdf.xacro (robot description, xacro)
@@ -27,3 +27,25 @@
   <xacro:panda_arm arm_id="$(arg an_an_id)" connected_to="base"  xyz="0.2336 0.515 1" rpy="0 0 ${-pi}" safety_distance="0.005"/>
   <!-- <xacro:hand arm_id="$(arg an_an_id)" rpy="0 0 ${-pi/4}" connected_to="$(arg an_an_id)_link8" safety_distance="0.005"/> -->
+  <link name="camera_mount">
+    <visual>
+      <origin xyz="0 0 0.23" rpy="0 0 0"/>
+      <geometry>
+        <box size="0.15 0.15 0.46" />
+      </geometry>
+      <material name="White">
+        <color rgba="1.0 1.0 1.0 1.0"/>
+      </material>
+    </visual>
+    <collision>
+      <origin xyz="0 0 0.23" rpy="0 0 0"/>
+      <geometry>
+        <box size="0.15 0.15 0.46" />
+      </geometry>
+    </collision>
+  </link>
+  <joint name="$(arg pan_pan_id)_d455_0_mount" type="fixed">
+     <origin xyz="0.15 -0.35 0.0" rpy="0 0 0"/>
+     <parent link="$(arg pan_pan_id)_link0"/>
+     <child link="camera_mount" />
+  </joint>
 </robot>

Commit message: add tf for base plate

File: franka_description/robots/dual_mars_arm.urdf.xacro (robot description, xacro)
@@ -29,4 +29,10 @@
   <xacro:panda_arm arm_id="$(arg an_an_id)" connected_to="base"  xyz="0.2301 0.5065 1.005" rpy="0 0 ${-pi}" safety_distance="0.005"/>
   <xacro:wsg_32_xacro name="$(arg an_an_id)_wsg" parent="$(arg an_an_id)_link8"  xyz="0 0 0.01" rpy="0 0 ${-pi/2}"/>
+  <link name="$(arg pan_pan_id)_base_plate" />
+  <joint name="$(arg pan_pan_id)_base_plate_joint" type="fixed">
+    <origin xyz="0.125855 -0.34327 -0.00525" rpy="0 0 0" />
+    <parent link="$(arg pan_pan_id)_link0" />
+    <child link="$(arg pan_pan_id)_base_plate" />
+  </joint>
   <!-- <xacro:hand arm_id="$(arg an_an_id)" rpy="0 0 ${-pi/4}" connected_to="$(arg an_an_id)_link8" safety_distance="0.005"/> -->
   <link name="camera_mount">

File: franka_description/robots/panda_arm.urdf.xacro (robot description, xacro)
@@ -12,8 +12,8 @@
     <xacro:panda_arm arm_id="$(arg arm_id)" safety_distance="0.03"/>
     <xacro:include filename="$(find wsg_32_description)/robots/wsg_32_description.urdf.xacro"/>
-    <xacro:wsg_32_xacro name="$(arg arm_id)_wsg" parent="$(arg arm_id)_link8"  xyz="0 0 0.01" rpy="0 0 -${pi/4}"/>
+    <xacro:wsg_32_xacro name="$(arg arm_id)_wsg" parent="$(arg arm_id)_link8"  xyz="0 0 0.01" rpy="0 0 -${pi/2}"/>
     <xacro:if value="$(arg hand)">
       <xacro:include filename="$(find franka_description)/robots/hand.xacro"/>
-      <xacro:hand arm_id="$(arg arm_id)" rpy="0 0 ${-pi/4}" connected_to="$(arg arm_id)_link8" safety_distance="0.03"/>
+      <xacro:hand arm_id="$(arg arm_id)" rpy="0 0 ${-pi/2}" connected_to="$(arg arm_id)_link8" safety_distance="0.03"/>
     </xacro:if>
     <link name="world" />
@@ -23,4 +23,10 @@
     </joint>
   </xacro:unless>
+  <link name="$(arg arm_id)_base_plate" />
+  <joint name="$(arg arm_id)_base_plate_joint" type="fixed">
+    <origin xyz="0.125855 -0.34327 -0.00525" rpy="0 0 0" />
+    <parent link="$(arg arm_id)_link0" />
+    <child link="$(arg arm_id)_base_plate" />
+  </joint>
   <xacro:if value="$(arg gazebo)">
     <xacro:arg name="xyz" default="0 0 0" />
